File: smd-led.sch (KiCad schematic (older format))
At the start: 54 parts, among them Q16 Q_NPN_BEC, Q17 Q_NPN_BEC, Q18 Q_NPN_BEC, Q19 Q_NPN_BEC

Commit message: add updated smd led footprint
Parts:
- R28, R31, R35, R38: Link (none) -> https://www.mouser.com/ProductDetail/652-CR0805FX-1002ELF
Changed lines of the file:
@@
 F 1 "68" H 2018 2155 50  0000 L CNN
 F 2 "Resistor_SMD:R_0805_2012Metric_Pad1.15x1.40mm_HandSolder" V 1990 2190 50  0001 C CNN
-F 3 "~" H 1950 2200 50  0001 C CNN
+F 3 "https://www.bourns.com/pdfs/chpreztr.pdf" H 1950 2200 50  0001 C CNN
+F 4 "" H 0   0   50  0001 C CNN "Link"
 	1    1950 2200
 	1    0    0    -1
@@
 F 1 "10k" H 1767 2445 50  0000 L CNN
 F 2 "Resistor_SMD:R_0805_2012Metric_Pad1.15x1.40mm_HandSolder" V 1740 2390 50  0001 C CNN
-F 3 "~" H 1700 2400 50  0001 C CNN
+F 3 "https://www.bourns.com/pdfs/chpreztr.pdf" H 1700 2400 50  0001 C CNN
+F 4 "https://www.mouser.com/ProductDetail/652-CR0805FX-1002ELF" H 0   0   50  0001 C CNN "Link"
 	1    1700 2400
 	-1   0    0    1
@@
 F 1 "68" H 2368 2155 50  0000 L CNN
 F 2 "Resistor_SMD:R_0805_2012Metric_Pad1.15x1.40mm_HandSolder" V 2340 2190 50  0001 C CNN
-F 3 "~" H 2300 2200 50  0001 C CNN
+F 3 "https://www.bourns.com/pdfs/chpreztr.pdf" H 2300 2200 50  0001 C CNN
+F 4 "" H 0   0   50  0001 C CNN "Link"
 	1    2300 2200
 	1    0    0    -1
@@
 F 1 "68" H 7268 2155 50  0000 L CNN
 F 2 "Resistor_SMD:R_0805_2012Metric_Pad1.15x1.40mm_HandSolder" V 7240 2190 50  0001 C CNN
-F 3 "~" H 7200 2200 50  0001 C CNN
+F 3 "https://www.bourns.com/pdfs/chpreztr.pdf" H 7200 2200 50  0001 C CNN
+F 4 "" H 0   0   50  0001 C CNN "Link"
 	1    7200 2200
 	1    0    0    -1
@@
 F 1 "10k" H 7018 2445 50  0000 L CNN
 F 2 "Resistor_SMD:R_0805_2012Metric_Pad1.15x1.40mm_HandSolder" V 6990 2390 50  0001 C CNN
-F 3 "~" H 6950 2400 50  0001 C CNN
+F 3 "https://www.bourns.com/pdfs/chpreztr.pdf" H 6950 2400 50  0001 C CNN
+F 4 "https://www.mouser.com/ProductDetail/652-CR0805FX-1002ELF" H 0   0   50  0001 C CNN "Link"
 	1    6950 2400
 	-1   0    0    1
@@
 F 1 "68" H 7618 2155 50  0000 L CNN
 F 2 "Resistor_SMD:R_0805_2012Metric_Pad1.15x1.40mm_HandSolder" V 7590 2190 50  0001 C CNN
-F 3 "~" H 7550 2200 50  0001 C CNN
+F 3 "https://www.bourns.com/pdfs/chpreztr.pdf" H 7550 2200 50  0001 C CNN
+F 4 "" H 0   0   50  0001 C CNN "Link"
 	1    7550 2200
 	1    0    0    -1
@@
 F 1 "68" H 9468 2155 50  0000 L CNN
 F 2 "Resistor_SMD:R_0805_2012Metric_Pad1.15x1.40mm_HandSolder" V 9440 2190 50  0001 C CNN
-F 3 "~" H 9400 2200 50  0001 C CNN
+F 3 "https://www.bourns.com/pdfs/chpreztr.pdf" H 9400 2200 50  0001 C CNN
+F 4 "" H 0   0   50  0001 C CNN "Link"
 	1    9400 2200
 	1    0    0    -1
@@
 F 1 "10k" H 9218 2445 50  0000 L CNN
 F 2 "Resistor_SMD:R_0805_2012Metric_Pad1.15x1.40mm_HandSolder" V 9190 2390 50  0001 C CNN
-F 3 "~" H 9150 2400 50  0001 C CNN
+F 3 "https://www.bourns.com/pdfs/chpreztr.pdf" H 9150 2400 50  0001 C CNN
+F 4 "https://www.mouser.com/ProductDetail/652-CR0805FX-1002ELF" H 0   0   50  0001 C CNN "Link"
 	1    9150 2400
 	-1   0    0    1
@@
 F 1 "68" H 9818 2155 50  0000 L CNN
 F 2 "Resistor_SMD:R_0805_2012Metric_Pad1.15x1.40mm_HandSolder" V 9790 2190 50  0001 C CNN
-F 3 "~" H 9750 2200 50  0001 C CNN
+F 3 "https://www.bourns.com/pdfs/chpreztr.pdf" H 9750 2200 50  0001 C CNN
+F 4 "" H 0   0   50  0001 C CNN "Link"
 	1    9750 2200
 	1    0    0    -1
@@
 F 1 "68" H 4468 2155 50  0000 L CNN
 F 2 "Resistor_SMD:R_0805_2012Metric_Pad1.15x1.40mm_HandSolder" V 4440 2190 50  0001 C CNN
-F 3 "~" H 4400 2200 50  0001 C CNN
+F 3 "https://www.bourns.com/pdfs/chpreztr.pdf" H 4400 2200 50  0001 C CNN
+F 4 "" H 0   0   50  0001 C CNN "Link"
 	1    4400 2200
 	1    0    0    -1
@@
 F 1 "10k" H 4218 2445 50  0000 L CNN
 F 2 "Resistor_SMD:R_0805_2012Metric_Pad1.15x1.40mm_HandSolder" V 4190 2390 50  0001 C CNN
-F 3 "~" H 4150 2400 50  0001 C CNN
+F 3 "https://www.bourns.com/pdfs/chpreztr.pdf" H 4150 2400 50  0001 C CNN
+F 4 "https://www.mouser.com/ProductDetail/652-CR0805FX-1002ELF" H 0   0   50  0001 C CNN "Link"
 	1    4150 2400
 	-1   0    0    1
@@
 F 1 "68" H 4818 2155 50  0000 L CNN
 F 2 "Resistor_SMD:R_0805_2012Metric_Pad1.15x1.40mm_HandSolder" V 4790 2190 50  0001 C CNN
-F 3 "~" H 4750 2200 50  0001 C CNN
+F 3 "https://www.bourns.com/pdfs/chpreztr.pdf" H 4750 2200 50  0001 C CNN
+F 4 "" H 0   0   50  0001 C CNN "Link"
 	1    4750 2200
 	1    0    0    -1
@@
 F 1 "68" H 5168 2155 50  0000 L CNN
 F 2 "Resistor_SMD:R_0805_2012Metric_Pad1.15x1.40mm_HandSolder" V 5140 2190 50  0001 C CNN
-F 3 "~" H 5100 2200 50  0001 C CNN
+F 3 "https://www.bourns.com/pdfs/chpreztr.pdf" H 5100 2200 50  0001 C CNN
+F 4 "" H 0   0   50  0001 C CNN "Link"
 	1    5100 2200
 	1    0    0    -1
@@
 F 1 "68" H 2018 5355 50  0000 L CNN
 F 2 "Resistor_SMD:R_0805_2012Metric_Pad1.15x1.40mm_HandSolder" V 1990 5390 50  0001 C CNN
-F 3 "~" H 1950 5400 50  0001 C CNN
+F 3 "https://www.bourns.com/pdfs/chpreztr.pdf" H 1950 5400 50  0001 C CNN
+F 4 "" H 0   0   50  0001 C CNN "Link"
 	1    1950 5400
 	1    0    0    -1
@@
 F 1 "68" H 2368 5355 50  0000 L CNN
 F 2 "Resistor_SMD:R_0805_2012Metric_Pad1.15x1.40mm_HandSolder" V 2340 5390 50  0001 C CNN
-F 3 "~" H 2300 5400 50  0001 C CNN
+F 3 "https://www.bourns.com/pdfs/chpreztr.pdf" H 2300 5400 50  0001 C CNN
+F 4 "" H 0   0   50  0001 C CNN "Link"
 	1    2300 5400
 	1    0    0    -1
@@
 F 1 "68" H 2718 5355 50  0000 L CNN
 F 2 "Resistor_SMD:R_0805_2012Metric_Pad1.15x1.40mm_HandSolder" V 2690 5390 50  0001 C CNN
-F 3 "~" H 2650 5400 50  0001 C CNN
+F 3 "https://www.bourns.com/pdfs/chpreztr.pdf" H 2650 5400 50  0001 C CNN
+F 4 "" H 0   0   50  0001 C CNN "Link"
 	1    2650 5400
 	1    0    0    -1
@@
 F 1 "68" H 3068 5355 50  0000 L CNN
 F 2 "Resistor_SMD:R_0805_2012Metric_Pad1.15x1.40mm_HandSolder" V 3040 5390 50  0001 C CNN
-F 3 "~" H 3000 5400 50  0001 C CNN
+F 3 "https://www.bourns.com/pdfs/chpreztr.pdf" H 3000 5400 50  0001 C CNN
+F 4 "" H 0   0   50  0001 C CNN "Link"
 	1    3000 5400
 	1    0    0    -1
@@
 F 1 "68" H 3418 5355 50  0000 L CNN
 F 2 "Resistor_SMD:R_0805_2012Metric_Pad1.15x1.40mm_HandSolder" V 3390 5390 50  0001 C CNN
-F 3 "~" H 3350 5400 50  0001 C CNN
+F 3 "https://www.bourns.com/pdfs/chpreztr.pdf" H 3350 5400 50  0001 C CNN
+F 4 "" H 0   0   50  0001 C CNN "Link"
 	1    3350 5400
 	1    0    0    -1
@@
 F 1 "68" H 3768 5355 50  0000 L CNN
 F 2 "Resistor_SMD:R_0805_2012Metric_Pad1.15x1.40mm_HandSolder" V 3740 5390 50  0001 C CNN
-F 3 "~" H 3700 5400 50  0001 C CNN
+F 3 "https://www.bourns.com/pdfs/chpreztr.pdf" H 3700 5400 50  0001 C CNN
+F 4 "" H 0   0   50  0001 C CNN "Link"
 	1    3700 5400
 	1    0    0    -1
@@
 F 1 "68" H 4918 5355 50  0000 L CNN
 F 2 "Resistor_SMD:R_0805_2012Metric_Pad1.15x1.40mm_HandSolder" V 4890 5390 50  0001 C CNN
-F 3 "~" H 4850 5400 50  0001 C CNN
+F 3 "https://www.bourns.com/pdfs/chpreztr.pdf" H 4850 5400 50  0001 C CNN
+F 4 "" H 0   0   50  0001 C CNN "Link"
 	1    4850 5400
 	1    0    0    -1
@@
 F 1 "68" H 5268 5355 50  0000 L CNN
 F 2 "Resistor_SMD:R_0805_2012Metric_Pad1.15x1.40mm_HandSolder" V 5240 5390 50  0001 C CNN
-F 3 "~" H 5200 5400 50  0001 C CNN
+F 3 "https://www.bourns.com/pdfs/chpreztr.pdf" H 5200 5400 50  0001 C CNN
+F 4 "" H 0   0   50  0001 C CNN "Link"
 	1    5200 5400
 	1    0    0    -1
@@
 F 1 "68" H 5618 5355 50  0000 L CNN
 F 2 "Resistor_SMD:R_0805_2012Metric_Pad1.15x1.40mm_HandSolder" V 5590 5390 50  0001 C CNN
-F 3 "~" H 5550 5400 50  0001 C CNN
+F 3 "https://www.bourns.com/pdfs/chpreztr.pdf" H 5550 5400 50  0001 C CNN
+F 4 "" H 0   0   50  0001 C CNN "Link"
 	1    5550 5400
 	1    0    0    -1
@@
 F 1 "68" H 5968 5355 50  0000 L CNN
 F 2 "Resistor_SMD:R_0805_2012Metric_Pad1.15x1.40mm_HandSolder" V 5940 5390 50  0001 C CNN
-F 3 "~" H 5900 5400 50  0001 C CNN
+F 3 "https://www.bourns.com/pdfs/chpreztr.pdf" H 5900 5400 50  0001 C CNN
+F 4 "" H 0   0   50  0001 C CNN "Link"
 	1    5900 5400
 	1    0    0    -1
@@
 F 1 "68" H 6318 5355 50  0000 L CNN
 F 2 "Resistor_SMD:R_0805_2012Metric_Pad1.15x1.40mm_HandSolder" V 6290 5390 50  0001 C CNN
-F 3 "~" H 6250 5400 50  0001 C CNN
+F 3 "https://www.bourns.com/pdfs/chpreztr.pdf" H 6250 5400 50  0001 C CNN
+F 4 "" H 0   0   50  0001 C CNN "Link"
 	1    6250 5400
 	1    0    0    -1
@@
 F 1 "68" H 6668 5355 50  0000 L CNN
 F 2 "Resistor_SMD:R_0805_2012Metric_Pad1.15x1.40mm_HandSolder" V 6640 5390 50  0001 C CNN
-F 3 "~" H 6600 5400 50  0001 C CNN
+F 3 "https://www.bourns.com/pdfs/chpreztr.pdf" H 6600 5400 50  0001 C CNN
+F 4 "" H 0   0   50  0001 C CNN "Link"
 	1    6600 5400
 	1    0    0    -1
@@
 F 1 "68" H 8418 5355 50  0000 L CNN
 F 2 "Resistor_SMD:R_0805_2012Metric_Pad1.15x1.40mm_HandSolder" V 8390 5390 50  0001 C CNN
-F 3 "~" H 8350 5400 50  0001 C CNN
+F 3 "https://www.bourns.com/pdfs/chpreztr.pdf" H 8350 5400 50  0001 C CNN
+F 4 "" H 0   0   50  0001 C CNN "Link"
 	1    8350 5400
 	1    0    0    -1
@@
 F 1 "68" H 9768 5355 50  0000 L CNN
 F 2 "Resistor_SMD:R_0805_2012Metric_Pad1.15x1.40mm_HandSolder" V 9740 5390 50  0001 C CNN
-F 3 "~" H 9700 5400 50  0001 C CNN
+F 3 "https://www.bourns.com/pdfs/chpreztr.pdf" H 9700 5400 50  0001 C CNN
+F 4 "" H 0   0   50  0001 C CNN "Link"
 	1    9700 5400
 	1    0    0    -1

Commit message: add io led specs
Parts:
- D10, D11, D12, D13, D14, D15, D16, D17, D18, D19, D20, D21, D22, D23, D24, D25, D26, D27, D5, D6, D7, D8, D9: Link https://www.mouser.com/ProductDetail/IN-S124BRUW -> (none)

Commit message: finish bom
Parts:
- D10, D11, D12, D13, D14, D15, D16, D17, D18, D19, D20, D21, D22, D23, D24, D25, D26, D27, D5, D6, D7, D8, D9: value LED -> Yellow; Link (none) -> https://www.mouser.com/ProductDetail/859-LTST-C230KSKT
- R29, R30, R32, R33, R34, R36, R37, R39, R40, R41, R42, R43, R44, R45, R46, R47, R48, R49, R50, R51, R52, R53, R54: value 68 -> 510; Link (none) -> https://www.mouser.com/ProductDetail/652-CR0805FX-5100ELF
